Commit message: fixed origin/rot in meshes and fixed urdf export

File: isaac_sim/assets/puzzlebot/urdf/puzzlebot_forklift2.urdf (robot description, URDF)
Before this commit: robot puzzlebot, 9 links, 8 joints
Links:
- removed link caster_wheel_link
- removed link chassis_link
- removed link left_wheel_link
- removed link right_wheel_link
- added link caster_wheel, mass 0.012; collision sphere radius=0.0065; visual mesh filename=../meshes2/puzzlebot_caster_wheel.obj
- added link chassis, mass 0.71; collision box size=0.2 0.16 0.06; visual mesh filename=../meshes2/puzzlebot_chassis_detailed.obj
- added link forks_link, mass 0.1; collision cylinder length=0.04 radius=0.05; visual mesh filename=../meshes/forks.obj
- added link inner_mast_link, mass 0.1; collision cylinder length=0.04 radius=0.05; visual mesh filename=../meshes2/inner_mast.stl
- added link left_wheel, mass 0.03; collision cylinder length=0.01 radius=0.05; visual mesh filename=../meshes/puzzlebot_wheel.obj
- added link outer_mast_link, mass 0.1; collision cylinder length=0.04 radius=0.05; visual mesh filename=../meshes2/outer_mast.obj
- added link right_wheel, mass 0.03; collision cylinder length=0.01 radius=0.05; visual mesh filename=../meshes/puzzlebot_wheel.obj
- link camera_color_optical_frame: mass 0.007 -> None; geometry 
Joints:
- added joint forks_joint: type prismatic, parent inner_mast_link, child forks_link, origin xyz=0.01 0 0 rpy=0 0 0, axis 0 0 1, limit lower=0.0 upper=0.20 effort=10 velocity=0.1
- added joint inner_mast_joint: type prismatic, parent outer_mast_link, child inner_mast_link, origin xyz=0 0 0 rpy=0 0 0, axis 0 0 1, limit lower=0.0 upper=0.20 effort=10 velocity=0.1
- added joint outer_mast_joint: type fixed, parent chassis, child outer_mast_link, origin xyz=0.12 0.0 -0.04 rpy=0 0 0
- joint base_link_to_chassis: child chassis_link -> chassis
- joint base_to_left_wheel: child left_wheel_link -> left_wheel; limit velocity=6 -> (none); origin xyz=0.05 0.09 0.0 rpy=0 0 0 -> xyz=0.05 0.095 0 rpy=0 0 0; parent chassis_link -> chassis
- joint base_to_right_wheel: child right_wheel_link -> right_wheel; limit velocity=6 -> (none); origin xyz=0.05 -0.09 0.0 rpy=0 0 0 -> xyz=0.05 -0.095 0 rpy=0 0 0; parent chassis_link -> chassis
- joint chassis_to_camera: origin xyz=0.1 0 0.07 rpy=0 0 0 -> xyz=0.0 0.0 0.12 rpy=0 0 0; parent chassis_link -> forks_link
- joint chassis_to_caster: child caster_wheel_link -> caster_wheel; parent chassis_link -> chassis
- joint chassis_to_lidar: parent chassis_link -> chassis
- joint optical_frame: origin xyz=0.02 0 0 rpy=-1.570796326794895 0 -1.570796326794895 -> xyz=0.0 0 0 rpy=-1.570796326794895 0 -1.570796326794895

File: isaac_sim/assets/puzzlebot/urdf/test3.urdf (robot description, URDF)
Before this commit: robot puzzlebot, 9 links, 8 joints
Links:
- added link fork_tip
- added link forks_link; visual mesh filename=../meshes3/forks.obj
- added link inner_mast_link; visual mesh filename=../meshes3/inner_mast.obj
- added link outer_mast_link; visual mesh filename=../meshes3/outer_mast.obj
- link camera_color_optical_frame: mass 0.007 -> None; geometry 
- link camera_link: geometry 
- link caster_wheel_link: geometry collision sphere radius=0.0065; visual mesh filename=../meshes3/puzzlebot_caster_wheel.obj
- link chassis_link: geometry collision box size=0.2 0.16 0.06; visual mesh filename=../meshes3/puzzlebot_chassis_detailed.obj
- link left_wheel_link: geometry collision cylinder length=0.01 radius=0.05; visual mesh filename=../meshes3/puzzlebot_wheel.obj
- link right_wheel_link: geometry collision cylinder length=0.01 radius=0.05; visual mesh filename=../meshes3/puzzlebot_wheel.obj
Joints:
- added joint forks_joint: type fixed, parent inner_mast_link, child forks_link, origin xyz=0 0 0 rpy=0 0 0
- added joint forks_to_tip: type fixed, parent forks_link, child fork_tip, origin xyz=0.109 0 0.0015 rpy=0 0 0
- added joint inner_mast_joint: type fixed, parent outer_mast_link, child inner_mast_link
- added joint outer_mast_joint: type fixed, parent chassis_link, child outer_mast_link, origin xyz=0.12 0.0 -0.04 rpy=0 0 0
- joint base_to_left_wheel: limit velocity=6 -> (none); origin xyz=0.05 0.09 0.0 rpy=0 0 0 -> xyz=0.05 0.095 0 rpy=0 0 0
- joint base_to_right_wheel: limit velocity=6 -> (none); origin xyz=0.05 -0.09 0.0 rpy=0 0 0 -> xyz=0.05 -0.095 0 rpy=0 0 0
- joint chassis_to_camera: origin xyz=0.1 0 0.07 rpy=0 0 0 -> xyz=0.0 0.0 0.1 rpy=0 0 0; parent chassis_link -> forks_link
- joint chassis_to_caster: origin xyz=-0.095 0.0 -0.0425 rpy=0 0 0 -> xyz=-0.095 0.0 -0.0435 rpy=0 0 0
- joint optical_frame: origin xyz=0.02 0 0 rpy=-1.570796326794895 0 -1.570796326794895 -> xyz=0.0 0 0 rpy=-1.570796326794895 0 -1.570796326794895

File: isaac_sim/assets/puzzlebot/urdf/test5.urdf (robot description, URDF)
Before this commit: robot puzzlebot, 9 links, 8 joints
Links:
- added link forks_link, mass 0.001; visual mesh filename=../meshes3/forks.obj
- link camera_color_optical_frame: mass 0.007 -> None; geometry 
- link camera_link: mass 0.007 -> None; geometry 
- link caster_wheel_link: geometry collision sphere radius=0.0065; visual mesh filename=../meshes3/puzzlebot_caster_wheel.obj
- link chassis_link: geometry collision box size=0.2 0.16 0.06; visual mesh filename=../meshes3/puzzlebot_chassis_detailed.obj
- link left_wheel_link: geometry collision cylinder length=0.01 radius=0.05; visual mesh filename=../meshes3/puzzlebot_wheel.obj
- link right_wheel_link: geometry collision cylinder length=0.01 radius=0.05; visual mesh filename=../meshes3/puzzlebot_wheel.obj
Joints:
- added joint forks_joint: type prismatic, parent chassis_link, child forks_link, origin xyz=0.12 0 0 rpy=0 0 0, axis 0 0 1, limit lower=0.0 upper=0.20 effort=10 velocity=0.1
- joint base_to_left_wheel: limit velocity=6 -> (none); origin xyz=0.05 0.09 0.0 rpy=0 0 0 -> xyz=0.05 0.095 0 rpy=0 0 0
- joint base_to_right_wheel: limit velocity=6 -> (none); origin xyz=0.05 -0.09 0.0 rpy=0 0 0 -> xyz=0.05 -0.095 0 rpy=0 0 0
- joint chassis_to_camera: origin xyz=0.1 0 0.07 rpy=0 0 0 -> xyz=0.0 0.0 0.1 rpy=0 0 0
- joint optical_frame: origin xyz=0.02 0 0 rpy=-1.570796326794895 0 -1.570796326794895 -> xyz=0.0 0 0 rpy=-1.570796326794895 0 -1.570796326794895

File: isaac_sim/assets/puzzlebot/urdf/test6.urdf (robot description, URDF)
Before this commit: robot puzzlebot, 9 links, 8 joints
Links:
- added link fork_tip_link
- added link forks_link, mass 0.001; collision box size=0.109 0.017 0.003; collision box size=0.109 0.017 0.003
- link camera_color_optical_frame: mass 0.007 -> None; geometry 
- link camera_link: mass 0.007 -> 0.001; geometry 
- link caster_wheel_link: geometry collision sphere radius=0.0065; visual mesh filename=../meshes3/puzzlebot_caster_wheel.obj
- link chassis_link: mass 0.71 -> 1.71; geometry collision box size=0.2 0.16 0.06; visual mesh filename=../meshes3/puzzlebot_chassis_detailed.obj
- link left_wheel_link: geometry collision cylinder length=0.01 radius=0.05; visual mesh filename=../meshes3/puzzlebot_wheel.obj
- link right_wheel_link: geometry collision cylinder length=0.01 radius=0.05; visual mesh filename=../meshes3/puzzlebot_wheel.obj
Joints:
- added joint forks_joint: type prismatic, parent chassis_link, child forks_link, origin xyz=0.12 0 -0.04 rpy=0 0 0, axis 0 0 1, limit lower=0.0 upper=0.2 effort=50 velocity=0.1
- added joint forks_to_tip: type fixed, parent forks_link, child fork_tip_link
- joint base_to_left_wheel: limit velocity=6 -> (none); origin xyz=0.05 0.09 0.0 rpy=0 0 0 -> xyz=0.05 0.095 0 rpy=0 0 0
- joint base_to_right_wheel: limit velocity=6 -> (none); origin xyz=0.05 -0.09 0.0 rpy=0 0 0 -> xyz=0.05 -0.095 0 rpy=0 0 0
- joint chassis_to_camera: origin xyz=0.1 0 0.07 rpy=0 0 0 -> xyz=0.0 0.0 0.1 rpy=0 0 0; parent chassis_link -> forks_link
- joint optical_frame: origin xyz=0.02 0 0 rpy=-1.570796326794895 0 -1.570796326794895 -> (none)

File: src/puzzlebot_description/urdf/materials.xacro (robot description, xacro)
@@ -25,3 +25,6 @@
     <color rgba="0.20 0.24 0.29 1.0"/>
   </material>
+  <material name="orange">
+    <color rgba="1.0 0.1 0.0 1.0"/>
+  </material>
 </robot>

File: src/puzzlebot_description/urdf/parameters.xacro (robot description, xacro)
@@ -15,7 +15,8 @@
 <!-- Distance from base link to the front edge of the chasis -->
   <xacro:property name="baselink_2_front"   value="0.09"/>
+  <xacro:property name="front_2_forklift"   value="0.03"/>
   <xacro:property name="caster_radius" value="0.0065"/>
   <xacro:property name="caster_mass"   value="0.012"/>
-  <!-- Posicionn relativa al chassis: atras y abajo -->
+  <!-- Posicionn relativa al chassis atras y abajo -->
   <xacro:property name="caster_x" value="-0.095"/>
   <xacro:property name="caster_y" value="0.0"/>
@@ -25,8 +26,8 @@
   <xacro:property name="camera_width"  value="0.01"/>
   <xacro:property name="camera_height" value="0.06"/>
-  <!-- camera position over the chassis-->
-  <xacro:property name="camera_x" value="0.08"/>
+  <!-- camera position over the chassis /OVER THE FORKS-->
+  <xacro:property name="camera_x" value="0.0"/>
   <xacro:property name="camera_y" value="0.0"/>
-  <xacro:property name="camera_z" value="0.07"/>
+  <xacro:property name="camera_z" value="0.10"/>
   <xacro:property name="lidar_mass"   value="0.1"/>
   <xacro:property name="lidar_x"      value="0.05"/>
@@ -34,23 +35,28 @@
   <xacro:property name="lidar_z"      value="0.115"/>
   <!-- fork position over the chassis FRONT-->
-  <xacro:property name="forks_x" value="${baselink_2_front + 0.064}"/>
+  <xacro:property name="forks_x" value="${baselink_2_front + front_2_forklift}"/>
   <xacro:property name="forks_y" value="0.0"/>
-  <xacro:property name="forks_z" value="-0.02"/>
-  <xacro:property name="forks_yaw" value="${PI}"/>
+  <xacro:property name="forks_z" value="-0.04"/>
+  <xacro:property name="forks_yaw" value= "0.0"/>
+<xacro:property name="mast_height"      value="0.169"/>
+<xacro:property name="mast_width"       value="0.0628"/>
+<xacro:property name="mast_thickness"   value="0.01"/>
+<xacro:property name="fork_length"      value="0.109"/>
+<xacro:property name="fork_width"       value="0.017"/>
+<xacro:property name="fork_thickness"   value="0.003"/>
+<xacro:property name="fork_separation"  value="0.045"/>  <!-- distance between 2 fingers -->
+<xacro:property name="inner_travel"     value="0.20"/>
+<xacro:property name="fork_travel"      value="0.20"/>
   <xacro:property name="mesh_chassis"
-    value="$(find puzzlebot_description)/meshes/chasis_detailed.stl"/>
+    value="$(find puzzlebot_description)/meshes/puzzlebot_chassis_detailed.obj"/>
   <xacro:property name="mesh_wheel"
-    value="$(find puzzlebot_description)/meshes/puzzlebot_wheel.stl"/>
-  <xacro:property name="mesh_camera"
-    value="$(find puzzlebot_description)/meshes/camera.stl"/>
-  <xacro:property name="mesh_lidar"
-    value="$(find puzzlebot_description)/meshes/lidar.stl"/>
+    value="$(find puzzlebot_description)/meshes/puzzlebot_wheel.obj"/>
   <xacro:property name="caster_wheel"
-    value="$(find puzzlebot_description)/meshes/puzzlebot_caster_wheel.stl"/>
+    value="$(find puzzlebot_description)/meshes/puzzlebot_caster_wheel.obj"/>
   <xacro:property name="mesh_forks"
-    value="$(find puzzlebot_description)/meshes/forks.stl"/>
+    value="$(find puzzlebot_description)/meshes/forks.obj"/>
   <xacro:property name="mesh_outer_mast"
-    value="$(find puzzlebot_description)/meshes/outer_mast.stl"/>
+    value="$(find puzzlebot_description)/meshes/outer_mast.obj"/>
   <xacro:property name="mesh_inner_mast"
-    value="$(find puzzlebot_description)/meshes/inner_mast.stl"/>
+    value="$(find puzzlebot_description)/meshes/inner_mast.obj"/>
 </robot>
