Commit message: fixed origin/rot in meshes and fixed urdf export

File: src/puzzlebot_description/urdf/puzzlebot.urdf.xacro (robot description, xacro)
@@ -19,12 +19,14 @@
   <joint name="${prefix}base_link_to_chassis" type="fixed">
     <parent link="${prefix}base_link"/>
-    <child  link="${prefix}chassis"/>
-    <origin xyz="0 0 0" rpy="0 0 0"/>
-  </joint>
-  <link name="${prefix}chassis">
-    <visual>
-      <origin xyz="0.050 0 0.1" rpy="${PI/2} 0 ${PI}"/>
-      <geometry>
+    <child  link="${prefix}chassis_link"/>
+    <origin xyz="0 0 0" rpy="0 0 0"/>
+  </joint>
+  <link name="${prefix}chassis_link">
+    <visual>
+      <origin xyz="0.04 0 -0.05" rpy="0 0 0"/>
+      <geometry>
+   <!-- <mesh filename="../meshes3/puzzlebot_chassis_detailed.obj"/> -->
         <mesh filename="file://${mesh_chassis}"/>
+       <!-- <mesh filename="../meshes3/puzzlebot_chassis_detailed.obj"/> -->
       </geometry>
       <material name="white"/>
@@ -46,8 +48,9 @@
     </inertial>
   </link>
-  <link name="${prefix}caster_wheel">
-    <visual>
-      <origin xyz="0 0 0" rpy="0 0 0"/>
-      <geometry>
+  <link name="${prefix}caster_wheel_link">
+    <visual>
+      <origin xyz="0 0 0" rpy="0 0 0"/>
+      <geometry>
+   <!-- <mesh filename="../meshes3/puzzlebot_caster_wheel.obj"/> -->
         <mesh filename="file://${caster_wheel}"/>
       </geometry>
@@ -67,52 +70,17 @@
   </link>
   <joint name="${prefix}chassis_to_caster" type="fixed">
-    <parent link="${prefix}chassis"/>
-    <child  link="${prefix}caster_wheel"/>
+    <parent link="${prefix}chassis_link"/>
+    <child  link="${prefix}caster_wheel_link"/>
     <origin xyz="${caster_x} ${caster_y} ${caster_z}" rpy="0 0 0"/>
   </joint>
-  <!-- RIGHT WHEEL -->
-  <link name="${prefix}right_wheel">
-    <visual>
-      <origin xyz="0 0 0" rpy="${PI/2} 0 0"/>
-      <geometry>
+  <!-- Left wheel -->
+  <link name="${prefix}left_wheel_link">
+    <visual>
+      <origin xyz="0 0 -0.046" rpy="0 0 0"/>
+      <geometry>
+   <!-- <mesh filename="../meshes3/puzzlebot_wheel.obj"/> -->
         <mesh filename="file://${mesh_wheel}"/>
       </geometry>
-      <material name="black"/>
-    </visual>
-    <collision>
-      <origin xyz="0 0 0" rpy="${PI/2} 0 0"/>
-      <geometry>
-        <cylinder length="${wheel_thickness}" radius="${wheel_radius}"/>
-      </geometry>
-    </collision>
-    <inertial>
-      <origin xyz="0 0 0" rpy="0 0 0"/>
-      <mass value="${wheel_mass}"/>
-      <!--
-        El cilindro tiene su eje en Z antes de la rotación visual.
-        La macro cylinder_inertia asume eje Z como eje de simetría.
-        Cuando el joint rota la rueda para que gire en Y, las inercias
-        se transforman automáticamente — no hay que hacer nada extra.
-      -->
-      <xacro:cylinder_inertia
-        m="${wheel_mass}"
-        r="${wheel_radius}"
-        l="${wheel_thickness}"/>
-    </inertial>
-  </link>
-  <joint name="${prefix}base_to_right_wheel" type="continuous">
-    <parent link="${prefix}chassis"/>
-    <child  link="${prefix}right_wheel"/>
-    <origin xyz="${wheel_x_offset} -${wheel_separation} 0" rpy="0 0 0"/>
-    <axis xyz="0 1 0"/>
-  </joint>
-  <!-- Left wheel -->
-  <link name="${prefix}left_wheel">
-    <visual>
-      <origin xyz="0 0 0" rpy="${PI/2} 0 0"/>
-      <geometry>
-        <mesh filename="file://${mesh_wheel}"/>
-      </geometry>
-      <material name="black"/>
+      <material name="orange"/>
     </visual>
     <collision>
@@ -132,24 +100,164 @@
   </link>
   <joint name="${prefix}base_to_left_wheel" type="continuous">
-    <parent link="${prefix}chassis"/>
-    <child  link="${prefix}left_wheel"/>
+    <parent link="${prefix}chassis_link"/>
+    <child  link="${prefix}left_wheel_link"/>
     <origin xyz="${wheel_x_offset} ${wheel_separation} 0" rpy="0 0 0"/>
     <axis xyz="0 1 0"/>
   </joint>
-<!-- camera -->
+  <!-- RIGHT WHEEL -->
+  <link name="${prefix}right_wheel_link">
+    <visual>
+      <origin xyz="0 0 -0.046" rpy="0 0 ${PI}"/>
+      <geometry>
+   <!-- <mesh filename="../meshes3/puzzlebot_wheel.obj"/> -->
+        <mesh filename="file://${mesh_wheel}"/>
+      </geometry>
+      <material name="orange"/>
+    </visual>
+    <collision>
+      <origin xyz="0 0 0" rpy="${PI/2} 0 0"/>
+      <geometry>
+        <cylinder length="${wheel_thickness}" radius="${wheel_radius}"/>
+      </geometry>
+    </collision>
+    <inertial>
+      <origin xyz="0 0 0" rpy="0 0 0"/>
+      <mass value="${wheel_mass}"/>
+      <xacro:cylinder_inertia
+        m="${wheel_mass}"
+        r="${wheel_radius}"
+        l="${wheel_thickness}"/>
+    </inertial>
+  </link>
+  <joint name="${prefix}base_to_right_wheel" type="continuous">
+    <parent link="${prefix}chassis_link"/>
+    <child  link="${prefix}right_wheel_link"/>
+    <origin xyz="${wheel_x_offset} -${wheel_separation} 0" rpy="0 0 0"/>
+    <axis xyz="0 1 0"/>
+  </joint>
+  <!-- lidar -->
+  <link name="${prefix}lidar_link">
+    <collision>
+      <origin xyz="0 0 0" rpy="0 0 0"/>
+      <geometry>
+        <cylinder length="0.04" radius="0.05"/>
+      </geometry>
+    </collision>
+    <inertial>
+      <origin xyz="0 0 0" rpy="0 0 0"/>
+      <mass value="${lidar_mass}"/>
+      <xacro:cylinder_inertia
+        m="${lidar_mass}"
+        r="0.05"
+        l="0.04"/>
+    </inertial>
+  </link>
+  <joint name="${prefix}chassis_to_lidar" type="fixed">
+    <parent link="${prefix}chassis_link"/>
+    <child  link="${prefix}lidar_link"/>
+    <origin xyz="${lidar_x} ${lidar_y} ${lidar_z}" rpy="0 0 ${PI}"/>
+  </joint>
+    <!-- outer_mast  -->
+<link name="${prefix}outer_mast_link">
+  <visual>
+    <origin xyz="0 0 0" rpy="0 0 0"/>
+    <geometry>
+    <!-- <mesh filename="../meshes3/outer_mast.obj"/> -->
+      <mesh filename="file://${mesh_outer_mast}"/>
+    </geometry>
+    <material name="black"/>
+  </visual>
+  <collision>
+    <origin xyz="0 0 ${mast_height/2}" rpy="0 0 0"/>
+    <geometry>
+      <box size="${mast_thickness} ${mast_width} ${mast_height}"/>
+    </geometry>
+  </collision>
+  <inertial>
+    <origin xyz="0 0 ${mast_height/2}" rpy="0 0 0"/>
+    <mass value="0.001"/>
+    <inertia ixx="1e-6" ixy="0" ixz="0" iyy="1e-6" iyz="0" izz="1e-6"/>
+  </inertial>
+</link>
+<joint name="${prefix}outer_mast_joint" type="fixed">
+  <parent link="${prefix}chassis_link"/>
+  <child  link="${prefix}outer_mast_link"/>
+  <origin xyz="${forks_x} ${forks_y} ${forks_z}" rpy="0 0 0"/>
+</joint>
+<link name="${prefix}inner_mast_link">
+  <visual>
+    <origin xyz="0 0 0" rpy="0 0 0"/>
+    <geometry>
+ <!-- <mesh filename="../meshes3/inner_mast.obj"/> -->
+      <mesh filename="file://${mesh_inner_mast}"/>
+    </geometry>
+    <material name="black"/>
+  </visual>
+  <collision>
+    <origin xyz="0 0 ${mast_height/2}" rpy="0 0 0"/>
+    <geometry>
+      <box size="${mast_thickness} ${mast_width} ${mast_height}"/>
+    </geometry>
+  </collision>
+  <inertial>
+    <origin xyz="0 0 ${mast_height/2}" rpy="0 0 0"/>
+    <mass value="0.001"/>
+    <inertia ixx="1e-6" ixy="0" ixz="0" iyy="1e-6" iyz="0" izz="1e-6"/>
+  </inertial>
+</link>
+<joint name="${prefix}inner_mast_joint" type="prismatic">
+  <parent link="${prefix}outer_mast_link"/>
+  <child  link="${prefix}inner_mast_link"/>
+  <origin xyz="0 0 0" rpy="0 0 0"/>
+  <axis xyz="0 0 1"/>
+  <limit lower="0.0" upper="${inner_travel}" effort="50" velocity="0.1"/>
+  <dynamics damping="1.0" friction="0.5"/>
+</joint>
+    <!-- FORKS -->
+<link name="${prefix}forks_link">
+  <visual>
+    <origin xyz="0 0 0" rpy="0 0 0"/>
+    <geometry>
+  <!-- <mesh filename="../meshes3/forks.obj"/> -->
+      <mesh filename="file://${mesh_forks}"/>
+    </geometry>
+    <material name="black"/>
+  </visual>
+  <!-- left finger -->
+  <collision>
+    <origin xyz="${fork_length/2} ${fork_separation/2} ${fork_thickness/2}" rpy="0 0 0"/>
+    <geometry>
+      <box size="${fork_length} ${fork_width} ${fork_thickness}"/>
+    </geometry>
+  </collision>
+  <!-- right finger -->
+  <collision>
+    <origin xyz="${fork_length/2} ${-fork_separation/2} ${fork_thickness/2}" rpy="0 0 0"/>
+    <geometry>
+      <box size="${fork_length} ${fork_width} ${fork_thickness}"/>
+    </geometry>
+  </collision>
+  <inertial>
+    <origin xyz="${fork_length/2} 0 0" rpy="0 0 0"/>
+    <mass value="0.001"/>
+    <inertia ixx="1e-6" ixy="0" ixz="0" iyy="1e-6" iyz="0" izz="1e-6"/>
+  </inertial>
+</link>
+<joint name="${prefix}forks_joint" type="prismatic">
+  <parent link="${prefix}inner_mast_link"/>
+  <child  link="${prefix}forks_link"/>
+  <origin xyz="0 0 0" rpy="0 0 0"/>
+  <axis xyz="0 0 1"/>
+  <limit lower="0.0" upper="${fork_travel}" effort="50" velocity="0.1"/>
+  <dynamics damping="1.0" friction="0.5"/>
+</joint>
+<link name="${prefix}fork_tip_link"/>
+<joint name="${prefix}forks_to_tip" type="fixed">
+  <parent link="${prefix}forks_link"/>
+  <child  link="${prefix}fork_tip_link"/>
+  <origin xyz="${fork_length} 0 ${fork_thickness/2}" rpy="0 0 0"/>
+</joint>
+  <!-- camera -->
   <link name="${prefix}camera_link">
-    <visual>
-      <origin xyz="0 0 0" rpy="0 0 ${PI}"/>
-      <geometry>
-        <!-- <mesh filename="file://${mesh_camera}"/> -->
-      </geometry>
-      <material name="blue"/>
-    </visual>
-    <collision>
-      <origin xyz="0 0 0" rpy="0 0 0"/>
-      <geometry>
-        <box size="${camera_length} ${camera_width} ${camera_height}"/>
-      </geometry>
-    </collision>
     <inertial>
       <origin xyz="0 0 0" rpy="0 0 0"/>
@@ -163,5 +271,5 @@
   </link>
   <joint name="${prefix}chassis_to_camera" type="fixed">
-    <parent link="${prefix}chassis"/>
+    <parent link="${prefix}forks_link"/>
     <child  link="${prefix}camera_link"/>
     <origin xyz="${camera_x} ${camera_y} ${camera_z}"
@@ -176,113 +284,3 @@
             rpy="-${PI/2} 0 -${PI/2}"/>
   </joint>
-  <!-- lidar -->
-  <link name="${prefix}lidar_link">
-    <visual>
-      <origin xyz="0.07 -0.013 -0.04" rpy="${PI/2} 0 0"/>
-      <geometry>
-        <!--<mesh filename="file://${mesh_lidar}"/> -->
-      </geometry>
-      <material name="dark_grey"/>
-    </visual>
-    <collision>
-      <origin xyz="0 0 0" rpy="0 0 0"/>
-      <geometry>
-        <cylinder length="0.04" radius="0.05"/>
-      </geometry>
-    </collision>
-    <inertial>
-      <origin xyz="0 0 0" rpy="0 0 0"/>
-      <mass value="${lidar_mass}"/>
-      <xacro:cylinder_inertia
-        m="${lidar_mass}"
-        r="0.05"
-        l="0.04"/>
-    </inertial>
-  </link>
-  <joint name="${prefix}chassis_to_lidar" type="fixed">
-    <parent link="${prefix}chassis"/>
-    <child  link="${prefix}lidar_link"/>
-    <origin xyz="${lidar_x} ${lidar_y} ${lidar_z}" rpy="0 0 ${PI}"/>
-  </joint>
-    <!-- outer_mast  -->
-  <link name="${prefix}outer_mast_link">
-    <visual>
-      <origin xyz="0.0 0.0 0.0" rpy="0 0 ${PI}"/>
-      <geometry>
-        <mesh filename="file://${mesh_outer_mast}"/>
-      </geometry>
-      <material name="black"/>
-    </visual>
-    <collision>
-      <origin xyz="0 0 0" rpy="0 0 0"/>
-      <geometry>
-        <cylinder length="0.04" radius="0.05"/>
-      </geometry>
-    </collision>
-    <inertial>
-      <origin xyz="0 0 0" rpy="0 0 0"/>
-      <mass value="0.1"/>
-      <inertia ixx="0.001" ixy="0" ixz="0" iyy="0.001" iyz="0" izz="0.001"/>
-    </inertial>
-  </link>
-  <joint name="${prefix}outer_mast_joint" type="fixed">
-    <parent link="${prefix}chassis"/>
-    <child  link="${prefix}outer_mast_link"/>
-    <origin xyz="${forks_x} ${forks_y} ${forks_z}" rpy="0 0 0"/>
-  </joint>
-  <link name="${prefix}inner_mast_link">
-    <visual>
-      <origin xyz="0.0 0.0 0.0" rpy="0 0 ${PI}"/>
-      <geometry>
-        <mesh filename="file://${mesh_inner_mast}"/>
-      </geometry>
-      <material name="black"/>
-    </visual>s
-    <collision>
-      <origin xyz="0 0 0" rpy="0 0 0"/>
-      <geometry>
-        <cylinder length="0.04" radius="0.05"/>
-      </geometry>
-    </collision>
-    <inertial>
-      <origin xyz="0 0 0" rpy="0 0 0"/>
-      <mass value="0.1"/>
-      <inertia ixx="0.001" ixy="0" ixz="0" iyy="0.001" iyz="0" izz="0.001"/>
-    </inertial>
-  </link>
-  <joint name="${prefix}inner_mast_joint" type="prismatic">
-    <parent link="${prefix}chassis"/>
-    <child  link="${prefix}inner_mast_link"/>
-    <origin xyz="${forks_x} ${forks_y} ${forks_z}" rpy="0 0 0"/>
-    <axis xyz="0 0 1"/>
-    <limit lower="0.0" upper="0.20" effort="10" velocity="0.1"/>
-  </joint>
-    <!-- FORKS -->
-  <link name="${prefix}forks_link">
-    <visual>
-      <origin xyz="0.0 0.0 0.0" rpy="0 0 ${PI}"/>
-      <geometry>
-        <mesh filename="file://${mesh_forks}"/>
-      </geometry>
-      <material name="black"/>
-    </visual>s
-    <collision>
-      <origin xyz="0 0 0" rpy="0 0 0"/>
-      <geometry>
-        <cylinder length="0.04" radius="0.05"/>
-      </geometry>
-    </collision>
-    <inertial>
-      <origin xyz="0 0 0" rpy="0 0 0"/>
-      <mass value="0.1"/>
-      <inertia ixx="0.001" ixy="0" ixz="0" iyy="0.001" iyz="0" izz="0.001"/>
-    </inertial>
-  </link>
-  <joint name="${prefix}forks_joint" type="prismatic">
-    <parent link="${prefix}chassis"/>
-    <child  link="${prefix}forks_link"/>
-    <origin xyz="${forks_x} ${forks_y} ${forks_z}" rpy="0 0 0"/>
-    <axis xyz="0 0 1"/>
-    <limit lower="0.0" upper="0.20" effort="10" velocity="0.1"/>
-  </joint>
 </robot>
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