Commit message: simulattion listens cmd_vel

File: isaac_sim/assets/puzzlebot/urdf/puzzlebot.urdf (robot description, URDF)
Before this commit: robot puzzlebot, 8 links, 7 joints
Links:
- removed link camera
- removed link caster_wheel
- removed link chassis
- removed link left_wheel
- removed link lidar
- removed link right_wheel
- added link camera_color_optical_frame, mass 0.007; collision box size=0.05 0.01 0.06
- added link camera_link, mass 0.007; collision box size=0.05 0.01 0.06
- added link caster_wheel_link, mass 0.012; collision sphere radius=0.0065; visual mesh filename=../meshes/puzzlebot_caster_wheel.obj
- added link chassis_link, mass 0.71; collision box size=0.2 0.16 0.06; visual mesh filename=../meshes/puzzlebot_chasis.obj
- added link left_wheel_link, mass 0.03; collision cylinder length=0.01 radius=0.05; visual mesh filename=../meshes/puzzlebot_wheel.obj
- added link lidar_link, mass 0.1; collision cylinder length=0.04 radius=0.05
- added link right_wheel_link, mass 0.03; collision cylinder length=0.01 radius=0.05; visual mesh filename=../meshes/puzzlebot_wheel.obj
Joints:
- added joint optical_frame: type fixed, parent camera_link, child camera_color_optical_frame, origin xyz=0.02 0 0 rpy=-1.570796326794895 0 -1.570796326794895
- joint base_link_to_chassis: child chassis -> chassis_link
- joint base_to_left_wheel: child left_wheel -> left_wheel_link; parent chassis -> chassis_link
- joint base_to_right_wheel: child right_wheel -> right_wheel_link; parent chassis -> chassis_link
- joint chassis_to_camera: child camera -> camera_link; origin xyz=0.09 0.0 0.048 rpy=1.570796326794895 3.14159265358979 1.570796326794895 -> xyz=0.1 0 0.07 rpy=0 0 0; parent chassis -> chassis_link
- joint chassis_to_caster: child caster_wheel -> caster_wheel_link; parent chassis -> chassis_link
- joint chassis_to_lidar: child lidar -> lidar_link; parent chassis -> chassis_link

Commit message: fixed sim urdf

File: isaac_sim/assets/puzzlebot/urdf/puzzlebot.urdf (robot description, URDF)
Before this commit: robot puzzlebot, 9 links, 8 joints
Links:
- link left_wheel_link: geometry collision cylinder length=0.01 radius=0.051; visual mesh filename=../meshes/puzzlebot_wheel.obj
- link right_wheel_link: geometry collision cylinder length=0.01 radius=0.051; visual mesh filename=../meshes/puzzlebot_wheel.obj
Joints:
- joint base_to_left_wheel: origin xyz=0.05 0.09 0 rpy=0 0 0 -> xyz=0.051 0.09 0 rpy=0 0 0
- joint base_to_right_wheel: origin xyz=0.05 -0.09 0 rpy=0 0 0 -> xyz=0.051 -0.09 0 rpy=0 0 0

Commit message: 1 version std alone sim works

File: isaac_sim/assets/puzzlebot/urdf/puzzlebot.urdf (robot description, URDF)
Before this commit: robot puzzlebot, 9 links, 8 joints
Links:
- link left_wheel_link: geometry collision cylinder length=0.01 radius=0.049; visual mesh filename=../meshes/puzzlebot_wheel.obj
- link right_wheel_link: geometry collision cylinder length=0.01 radius=0.049; visual mesh filename=../meshes/puzzlebot_wheel.obj

Commit message: frctin cfg in isaac

File: isaac_sim/assets/puzzlebot/urdf/puzzlebot.urdf (robot description, URDF)
Before this commit: robot puzzlebot, 9 links, 8 joints
Links:
- link left_wheel_link: geometry collision cylinder length=0.01 radius=0.051; visual mesh filename=../meshes/puzzlebot_wheel.obj
- link right_wheel_link: geometry collision cylinder length=0.01 radius=0.051; visual mesh filename=../meshes/puzzlebot_wheel.obj

Commit message: cleaned isaac dir

File: isaac_sim/assets/puzzlebot/urdf/puzzlebot.urdf (robot description, URDF)
Before this commit: robot puzzlebot, 9 links, 8 joints
Links:
- link left_wheel_link: geometry collision cylinder length=0.01 radius=0.05; visual mesh filename=../meshes/puzzlebot_wheel.obj
- link right_wheel_link: geometry collision cylinder length=0.01 radius=0.05; visual mesh filename=../meshes/puzzlebot_wheel.obj
Joints:
- joint base_to_left_wheel: limit (none) -> velocity=6; origin xyz=0.051 0.09 0 rpy=0 0 0 -> xyz=0.05 0.09 0.0 rpy=0 0 0
- joint base_to_right_wheel: limit (none) -> velocity=6; origin xyz=0.051 -0.09 0 rpy=0 0 0 -> xyz=0.05 -0.09 0.0 rpy=0 0 0

File: src/puzzlebot_description/urdf/parameters.xacro (robot description, xacro)
@@ -6,9 +6,9 @@
   <xacro:property name="chassis_height" value="0.06"/>
   <xacro:property name="chassis_mass"   value="0.710"/>
-  <xacro:property name="wheel_radius"    value="0.051"/>
+  <xacro:property name="wheel_radius"    value="0.05"/>
   <xacro:property name="wheel_thickness" value="0.01"/>
   <xacro:property name="wheel_mass"      value="0.03"/>
   <!-- Distancia desde el centro del chassis al centro de cada rueda en Y -->
-  <xacro:property name="wheel_separation" value="0.09"/>
+  <xacro:property name="wheel_separation" value="0.095"/>
   <!-- Offset en X: las ruedas no están centradas, van ligeramente adelante -->
   <xacro:property name="wheel_x_offset"   value="0.05"/>

Commit message: mesh and xacro for forklift

File: isaac_sim/assets/puzzlebot/urdf/puzzlebot.urdf (robot description, URDF)
Before this commit: robot puzzlebot, 9 links, 8 joints
Links:
- link chassis_link: geometry collision box size=0.2 0.16 0.06; visual mesh filename=../meshes/puzzlebot_chassis_detailed.obj

File: src/puzzlebot_description/urdf/parameters.xacro (robot description, xacro)
@@ -13,7 +13,9 @@
   <!-- Offset en X: las ruedas no están centradas, van ligeramente adelante -->
   <xacro:property name="wheel_x_offset"   value="0.05"/>
+<!-- Distance from base link to the front edge of the chasis -->
+  <xacro:property name="baselink_2_front"   value="0.09"/>
   <xacro:property name="caster_radius" value="0.0065"/>
   <xacro:property name="caster_mass"   value="0.012"/>
-  <!-- Posición relativa al chassis: atrás y abajo -->
+  <!-- Posicionn relativa al chassis: atras y abajo -->
   <xacro:property name="caster_x" value="-0.095"/>
   <xacro:property name="caster_y" value="0.0"/>
@@ -31,6 +33,11 @@
   <xacro:property name="lidar_y"      value="0.0"/>
   <xacro:property name="lidar_z"      value="0.115"/>
+  <!-- fork position over the chassis FRONT-->
+  <xacro:property name="forks_x" value="${baselink_2_front + 0.064}"/>
+  <xacro:property name="forks_y" value="0.0"/>
+  <xacro:property name="forks_z" value="-0.02"/>
+  <xacro:property name="forks_yaw" value="${PI}"/>
   <xacro:property name="mesh_chassis"
-    value="$(find puzzlebot_description)/meshes/chassis.stl"/>
+    value="$(find puzzlebot_description)/meshes/chasis_detailed.stl"/>
   <xacro:property name="mesh_wheel"
     value="$(find puzzlebot_description)/meshes/puzzlebot_wheel.stl"/>
@@ -41,3 +48,9 @@
   <xacro:property name="caster_wheel"
     value="$(find puzzlebot_description)/meshes/puzzlebot_caster_wheel.stl"/>
+  <xacro:property name="mesh_forks"
+    value="$(find puzzlebot_description)/meshes/forks.stl"/>
+  <xacro:property name="mesh_outer_mast"
+    value="$(find puzzlebot_description)/meshes/outer_mast.stl"/>
+  <xacro:property name="mesh_inner_mast"
+    value="$(find puzzlebot_description)/meshes/inner_mast.stl"/>
 </robot>

File: src/puzzlebot_description/urdf/puzzlebot.urdf.xacro (robot description, xacro)
@@ -205,3 +205,84 @@
     <origin xyz="${lidar_x} ${lidar_y} ${lidar_z}" rpy="0 0 ${PI}"/>
   </joint>
+    <!-- outer_mast  -->
+  <link name="${prefix}outer_mast_link">
+    <visual>
+      <origin xyz="0.0 0.0 0.0" rpy="0 0 ${PI}"/>
+      <geometry>
+        <mesh filename="file://${mesh_outer_mast}"/>
+      </geometry>
+      <material name="black"/>
+    </visual>
+    <collision>
+      <origin xyz="0 0 0" rpy="0 0 0"/>
+      <geometry>
+        <cylinder length="0.04" radius="0.05"/>
+      </geometry>
+    </collision>
+    <inertial>
+      <origin xyz="0 0 0" rpy="0 0 0"/>
+      <mass value="0.1"/>
+      <inertia ixx="0.001" ixy="0" ixz="0" iyy="0.001" iyz="0" izz="0.001"/>
+    </inertial>
+  </link>
+  <joint name="${prefix}outer_mast_joint" type="fixed">
+    <parent link="${prefix}chassis"/>
+    <child  link="${prefix}outer_mast_link"/>
+    <origin xyz="${forks_x} ${forks_y} ${forks_z}" rpy="0 0 0"/>
+  </joint>
+  <link name="${prefix}inner_mast_link">
+    <visual>
+      <origin xyz="0.0 0.0 0.0" rpy="0 0 ${PI}"/>
+      <geometry>
+        <mesh filename="file://${mesh_inner_mast}"/>
+      </geometry>
+      <material name="black"/>
+    </visual>s
+    <collision>
+      <origin xyz="0 0 0" rpy="0 0 0"/>
+      <geometry>
+        <cylinder length="0.04" radius="0.05"/>
+      </geometry>
+    </collision>
+    <inertial>
+      <origin xyz="0 0 0" rpy="0 0 0"/>
+      <mass value="0.1"/>
+      <inertia ixx="0.001" ixy="0" ixz="0" iyy="0.001" iyz="0" izz="0.001"/>
+    </inertial>
+  </link>
+  <joint name="${prefix}inner_mast_joint" type="prismatic">
+    <parent link="${prefix}chassis"/>
+    <child  link="${prefix}inner_mast_link"/>
+    <origin xyz="${forks_x} ${forks_y} ${forks_z}" rpy="0 0 0"/>
+    <axis xyz="0 0 1"/>
+    <limit lower="0.0" upper="0.20" effort="10" velocity="0.1"/>
+  </joint>
+    <!-- FORKS -->
+  <link name="${prefix}forks_link">
+    <visual>
+      <origin xyz="0.0 0.0 0.0" rpy="0 0 ${PI}"/>
+      <geometry>
+        <mesh filename="file://${mesh_forks}"/>
+      </geometry>
+      <material name="black"/>
+    </visual>s
+    <collision>
+      <origin xyz="0 0 0" rpy="0 0 0"/>
+      <geometry>
+        <cylinder length="0.04" radius="0.05"/>
+      </geometry>
+    </collision>
+    <inertial>
+      <origin xyz="0 0 0" rpy="0 0 0"/>
+      <mass value="0.1"/>
+      <inertia ixx="0.001" ixy="0" ixz="0" iyy="0.001" iyz="0" izz="0.001"/>
+    </inertial>
+  </link>
+  <joint name="${prefix}forks_joint" type="prismatic">
+    <parent link="${prefix}chassis"/>
+    <child  link="${prefix}forks_link"/>
+    <origin xyz="${forks_x} ${forks_y} ${forks_z}" rpy="0 0 0"/>
+    <axis xyz="0 0 1"/>
+    <limit lower="0.0" upper="0.20" effort="10" velocity="0.1"/>
+  </joint>
 </robot>

Commit message: scene in isaac updated as real

File: isaac_sim/assets/puzzlebot/urdf/puzzlebot.urdf (robot description, URDF)
Before this commit: robot puzzlebot, 9 links, 8 joints
Links:
- removed link lidar_link
- added link laser, mass 0.1; collision cylinder length=0.04 radius=0.05
Joints:
- joint chassis_to_lidar: origin xyz=0.05 0.0 0.115 rpy=0 0 3.14159265358979 -> xyz=0.03 0.0 0.115 rpy=0 0 3.14159265358979

File: isaac_sim/assets/puzzlebot/urdf/test5.urdf (robot description, URDF)
Before this commit: robot puzzlebot, 10 links, 9 joints
Links:
- removed link lidar_link
- added link laser, mass 0.1; collision cylinder length=0.04 radius=0.05
Joints:
- joint chassis_to_camera: origin xyz=0.0 0.0 0.1 rpy=0 0 0 -> xyz=0.09 0.0 0.1 rpy=0 0 0
- joint chassis_to_lidar: child lidar_link -> laser; origin xyz=0.05 0.0 0.115 rpy=0 0 3.14159265358979 -> xyz=0.03 0.0 0.115 rpy=0 0 3.14159265358979
