Commit message: forklift and robot urdf complete

File: isaac_sim/assets/puzzlebot/urdf/test5.urdf (robot description, URDF)
Before this commit: robot puzzlebot, 10 links, 9 joints
Links:
- added link inner_mast_link, mass 0.08; collision box size=0.012 0.0561 0.16; visual mesh filename=../meshes3/inner_mast.obj
- added link outer_mast_link, mass 0.1; collision box size=0.025 0.0621 0.1698; visual mesh filename=../meshes3/outer_mast.obj
- link forks_link: mass 0.001 -> 0.15; geometry collision box size=0.0112 0.1087 0.0417; collision box size=0.1053 0.0184 0.004
- link laser: geometry collision cylinder length=0.044 radius=0.0355
Joints:
- added joint inner_mast_joint: type prismatic, parent outer_mast_link, child inner_mast_link, origin xyz=0 0 0 rpy=0 0 0, axis 0 0 1, limit lower=-0.05 upper=0.25 effort=10 velocity=0.05
- added joint outer_mast_joint: type fixed, parent chassis_link, child outer_mast_link, origin xyz=0.12 0.0 -0.04 rpy=0 0 0
- joint forks_joint: axis 0 0 1 -> (none); limit lower=0.0 upper=0.20 effort=10 velocity=0.1 -> (none); origin xyz=0.12 0 0 rpy=0 0 0 -> xyz=0 0 0.04 rpy=0 0 0; parent chassis_link -> inner_mast_link; type prismatic -> fixed
