Commit message: deleted old files

File: isaac_sim/assets/puzzlebot/urdf/puzzlebot_forklift_nw.urdf (robot description, URDF)
Before this commit: robot puzzlebot, 12 links, 11 joints
Links:
- removed link caster_wheel_link
- removed link chassis_link
- removed link laser
- removed link left_wheel_link
- removed link right_wheel_link
- added link caster_wheel, mass 0.012; collision sphere radius=0.0065; visual mesh filename=../meshes2/puzzlebot_caster_wheel.obj
- added link chassis, mass 0.71; collision box size=0.2 0.16 0.06; visual mesh filename=../meshes2/puzzlebot_chassis_detailed.obj
- added link left_wheel, mass 0.03; collision cylinder length=0.01 radius=0.05; visual mesh filename=../meshes2/puzzlebot_wheel.obj
- added link lidar_link, mass 0.1; collision cylinder length=0.04 radius=0.05
- added link right_wheel, mass 0.03; collision cylinder length=0.01 radius=0.05; visual mesh filename=../meshes2/puzzlebot_wheel.obj
- link camera_link: mass None -> 0.007; geometry collision box size=0.05 0.01 0.06
- link forks_link: mass 0.15 -> 0.1; geometry collision cylinder length=0.04 radius=0.05; visual mesh filename=../meshes/forks.obj
- link inner_mast_link: mass 0.08 -> 0.1; geometry collision cylinder length=0.04 radius=0.05; visual mesh filename=../meshes/inner_mast.stl
- link outer_mast_link: geometry collision cylinder length=0.04 radius=0.05; visual mesh filename=../meshes2/outer_mast.obj
Joints:
- joint base_link_to_chassis: child chassis_link -> chassis
- joint base_to_left_wheel: child left_wheel_link -> left_wheel; parent chassis_link -> chassis
- joint base_to_right_wheel: child right_wheel_link -> right_wheel; parent chassis_link -> chassis
- joint chassis_to_camera: origin xyz=0.09 0.0 0.1 rpy=0 0 0 -> xyz=0.0 0.0 0.12 rpy=0 0 0; parent chassis_link -> forks_link
- joint chassis_to_caster: child caster_wheel_link -> caster_wheel; parent chassis_link -> chassis
- joint chassis_to_lidar: child laser -> lidar_link; origin xyz=0.03 0.0 0.115 rpy=0 0 3.14159265358979 -> xyz=0.05 0.0 0.115 rpy=0 0 3.14159265358979; parent chassis_link -> chassis
- joint forks_joint: axis (none) -> 0 0 1; limit (none) -> lower=0.0 upper=0.20 effort=10 velocity=0.1; origin xyz=0 0 0.04 rpy=0 0 0 -> xyz=0.01 0 0 rpy=0 0 0; type fixed -> prismatic
- joint inner_mast_joint: limit lower=-0.05 upper=0.25 effort=10 velocity=0.05 -> lower=0.0 upper=0.20 effort=10 velocity=0.1
- joint outer_mast_joint: parent chassis_link -> chassis
