Commit message: mass almost 0 to cam and 2 dof for fork

File: isaac_sim/assets/puzzlebot/urdf/puzzlebot_forklift.urdf (robot description, URDF)
Before this commit: robot puzzlebot, 12 links, 11 joints
Links:
- removed link caster_wheel
- removed link chassis
- removed link left_wheel
- removed link lidar_link
- removed link right_wheel
- added link caster_wheel_link, mass 0.012; collision sphere radius=0.0065; visual mesh filename=../meshes3/puzzlebot_caster_wheel.obj
- added link chassis_link, mass 0.71; collision box size=0.2 0.16 0.06; visual mesh filename=../meshes3/puzzlebot_chassis_detailed.obj
- added link laser, mass 0.1; collision cylinder length=0.044 radius=0.0355
- added link left_wheel_link, mass 0.03; collision cylinder length=0.01 radius=0.05; visual mesh filename=../meshes3/puzzlebot_wheel.obj
- added link right_wheel_link, mass 0.03; collision cylinder length=0.01 radius=0.05; visual mesh filename=../meshes3/puzzlebot_wheel.obj
- link camera_color_optical_frame: mass None -> 0.0001
- link camera_link: geometry 
- link forks_link: mass 0.1 -> 0.15; geometry collision box size=0.0112 0.1087 0.0417; collision box size=0.1053 0.0184 0.004
- link inner_mast_link: mass 0.1 -> 0.08; geometry collision box size=0.012 0.0561 0.16; visual mesh filename=../meshes3/inner_mast.obj
- link outer_mast_link: geometry collision box size=0.025 0.0621 0.1698; visual mesh filename=../meshes3/outer_mast.obj
Joints:
- joint base_link_to_chassis: child chassis -> chassis_link
- joint base_to_left_wheel: child left_wheel -> left_wheel_link; parent chassis -> chassis_link
- joint base_to_right_wheel: child right_wheel -> right_wheel_link; parent chassis -> chassis_link
- joint chassis_to_camera: origin xyz=0.0 0.0 0.12 rpy=0 0 0 -> xyz=0.09 0.0 0.1 rpy=0 0 0
- joint chassis_to_caster: child caster_wheel -> caster_wheel_link; parent chassis -> chassis_link
- joint chassis_to_lidar: child lidar_link -> laser; origin xyz=0.05 0.0 0.115 rpy=0 0 3.14159265358979 -> xyz=0.03 0.0 0.115 rpy=0 0 3.14159265358979; parent chassis -> chassis_link
- joint forks_joint: limit lower=0.0 upper=0.20 effort=10 velocity=0.1 -> lower=-0.01 upper=0.10 effort=10 velocity=0.05; origin xyz=0.01 0 0 rpy=0 0 0 -> xyz=0 0 0.04 rpy=0 0 0
- joint inner_mast_joint: limit lower=0.0 upper=0.20 effort=10 velocity=0.1 -> lower=-0.04 upper=0.25 effort=10 velocity=0.05
- joint outer_mast_joint: parent chassis -> chassis_link

Commit message: changed tf in camera to fork

File: isaac_sim/assets/puzzlebot/urdf/puzzlebot_forklift.urdf (robot description, URDF)
Before this commit: robot puzzlebot, 12 links, 11 joints
Joints:
- joint chassis_to_camera: origin xyz=0.09 0.0 0.1 rpy=0 0 0 -> xyz=0.015 0.0 0.1 rpy=0 0 0

File: src/puzzlebot_description/urdf/parameters.xacro (robot description, xacro)
@@ -13,7 +13,4 @@
   <!-- Offset en X: las ruedas no están centradas, van ligeramente adelante -->
   <xacro:property name="wheel_x_offset"   value="0.05"/>
-<!-- Distance from base link to the front edge of the chasis -->
-  <xacro:property name="baselink_2_front"   value="0.09"/>
-  <xacro:property name="front_2_forklift"   value="0.05"/>
   <xacro:property name="caster_radius" value="0.0065"/>
   <xacro:property name="caster_mass"   value="0.012"/>
@@ -26,27 +23,49 @@
   <xacro:property name="camera_width"  value="0.01"/>
   <xacro:property name="camera_height" value="0.06"/>
-  <!-- camera position over the chassis /OVER THE FORKS-->
-  <xacro:property name="camera_x" value="0.01"/>
+  <!-- camera pose in forks_link, so it rides up and down with the carriage -->
+  <xacro:property name="camera_x" value="0.015"/>
   <xacro:property name="camera_y" value="0.0"/>
-  <xacro:property name="camera_z" value="0.15"/>
-  <!--<xacro:property name="forks_z" value="0.005"-->
+  <xacro:property name="camera_z" value="0.1"/>
+  <!-- a link without <inertial> gets 1 kg in PhysX, so even the optical frame carries a token mass -->
+  <xacro:property name="optical_mass" value="0.0001"/>
+  <xacro:property name="optical_inertia" value="1e-9"/>
   <xacro:property name="lidar_mass"   value="0.1"/>
   <xacro:property name="lidar_x"      value="0.03"/>
   <xacro:property name="lidar_y"      value="0.0"/>
   <xacro:property name="lidar_z"      value="0.115"/>
-  <!-- fork position over the baseFRONT FRONT-->
-  <xacro:property name="forks_x" value="${baselink_2_front + front_2_forklift}"/>
-  <xacro:property name="forks_y" value="0.0"/>
-  <xacro:property name="forks_z" value="0.005"/>
-  <xacro:property name="forks_yaw" value= "0.0"/>
-<xacro:property name="mast_height"      value="0.169"/>
-<xacro:property name="mast_width"       value="0.0628"/>
-<xacro:property name="mast_thickness"   value="0.01"/>
-<xacro:property name="fork_length"      value="0.109"/>
-<xacro:property name="fork_width"       value="0.017"/>
-<xacro:property name="fork_thickness"   value="0.003"/>
-<xacro:property name="fork_separation"  value="0.045"/>  <!-- distance between 2 fingers -->
-<xacro:property name="inner_travel"     value="0.20"/>
-<xacro:property name="fork_travel"      value="0.20"/>
+  <!-- sized from the lidar head in the chassis mesh; expressed in the laser frame, which is yawed 180 deg -->
+  <xacro:property name="lidar_radius" value="0.0355"/>
+  <xacro:property name="lidar_length" value="0.044"/>
+  <xacro:property name="lidar_cx"     value="-0.0095"/>
+  <xacro:property name="lidar_cz"     value="-0.014"/>
+  <!-- outer mast: fixed to the chassis_link -->
+  <xacro:property name="outer_mast_x" value="0.12"/>
+  <xacro:property name="outer_mast_y" value="0.0"/>
+  <xacro:property name="outer_mast_z" value="-0.04"/>
+  <xacro:property name="outer_mast_mass" value="0.1"/>
+  <xacro:property name="outer_mast_visual_x" value="0.01"/>
+  <xacro:property name="outer_mast_box" value="0.025 0.0621 0.1698"/>
+  <xacro:property name="outer_mast_com" value="-0.0032 -0.0003 0.0856"/>
+  <!-- inner mast: smaller cross section so it nests inside the outer one -->
+  <xacro:property name="inner_mast_mass" value="0.08"/>
+  <xacro:property name="inner_mast_visual_z" value="0.023"/>
+  <xacro:property name="inner_mast_box" value="0.012 0.0561 0.16"/>
+  <xacro:property name="inner_mast_com" value="-0.0078 -0.0005 0.1125"/>
+  <xacro:property name="inner_lower" value="-0.04"/>
+  <xacro:property name="inner_upper" value="0.25"/>
+  <!-- forks (carriage). 0.04 cancels the outer mast drop so the forks keep their height at rest -->
+  <xacro:property name="forks_z" value="0.04"/>
+  <xacro:property name="forks_mass" value="0.15"/>
+  <xacro:property name="forks_com" value="0.0178 0.0097 0.0196"/>
+  <xacro:property name="forks_lower" value="-0.01"/>
+  <xacro:property name="forks_upper" value="0.10"/>
+  <xacro:property name="back_origin"  value="0.0056 0.01255 0.025"/>
+  <xacro:property name="back_size"    value="0.0112 0.1087 0.0417"/>
+  <xacro:property name="tine_l_origin" value="0.0578 0.0231 0.002"/>
+  <xacro:property name="tine_r_origin" value="0.0578 -0.0224 0.002"/>
+  <xacro:property name="tine_size"    value="0.1053 0.0184 0.004"/>
+  <!-- front end of the tines, used as the pallet-engaging frame -->
+  <xacro:property name="fork_tip_x" value="0.1105"/>
+  <xacro:property name="fork_tip_z" value="0.002"/>
   <xacro:property name="mesh_chassis"
     value="$(find puzzlebot_description)/meshes/puzzlebot_chassis_detailed.obj"/>

Commit message: Raise the lidar and lower the masts so they no longer block the scan
Lidar 1.5 cm higher, outer and inner mast meshes resting 0.8 cm above the
chassis bottom. Fork, camera and tip keep their rest height and the stack
travel stays [-0.05, 0.35] by shifting the joint origins and limits. Applied to
the xacro and to the Isaac URDF.

File: isaac_sim/assets/puzzlebot/urdf/puzzlebot_forklift.urdf (robot description, URDF)
Before this commit: robot puzzlebot, 12 links, 11 joints
Joints:
- joint chassis_to_lidar: origin xyz=0.03 0.0 0.115 rpy=0 0 3.14159265358979 -> xyz=0.03 0.0 0.13 rpy=0 0 3.14159265358979
- joint forks_joint: limit lower=-0.01 upper=0.10 effort=10 velocity=0.05 -> lower=-0.044 upper=0.0664 effort=10 velocity=0.05; origin xyz=0 0 0.04 rpy=0 0 0 -> xyz=0 0 0.0736 rpy=0 0 0
- joint inner_mast_joint: limit lower=-0.04 upper=0.25 effort=10 velocity=0.05 -> lower=-0.006 upper=0.2836 effort=10 velocity=0.05; origin xyz=0 0 0 rpy=0 0 0 -> xyz=0 0 -0.0318 rpy=0 0 0
- joint outer_mast_joint: origin xyz=0.12 0.0 -0.04 rpy=0 0 0 -> xyz=0.12 0.0 -0.0418 rpy=0 0 0

File: src/puzzlebot_description/urdf/parameters.xacro (robot description, xacro)
@@ -33,5 +33,5 @@
   <xacro:property name="lidar_x"      value="0.03"/>
   <xacro:property name="lidar_y"      value="0.0"/>
-  <xacro:property name="lidar_z"      value="0.115"/>
+  <xacro:property name="lidar_z"      value="0.13"/>
   <!-- sized from the lidar head in the chassis mesh; expressed in the laser frame, which is yawed 180 deg -->
   <xacro:property name="lidar_radius" value="0.0355"/>
@@ -42,5 +42,6 @@
   <xacro:property name="outer_mast_x" value="0.12"/>
   <xacro:property name="outer_mast_y" value="0.0"/>
-  <xacro:property name="outer_mast_z" value="-0.04"/>
+  <!-- mesh bottom sits 0.8 cm above the chassis mesh bottom (z -0.0491 in the chassis frame) -->
+  <xacro:property name="outer_mast_z" value="-0.0418"/>
   <xacro:property name="outer_mast_mass" value="0.1"/>
   <xacro:property name="outer_mast_visual_x" value="0.01"/>
@@ -52,12 +53,15 @@
   <xacro:property name="inner_mast_box" value="0.012 0.0561 0.16"/>
   <xacro:property name="inner_mast_com" value="-0.0078 -0.0005 0.1125"/>
-  <xacro:property name="inner_lower" value="-0.04"/>
-  <xacro:property name="inner_upper" value="0.25"/>
-  <!-- forks (carriage). 0.04 cancels the outer mast drop so the forks keep their height at rest -->
-  <xacro:property name="forks_z" value="0.04"/>
+  <!-- inner mesh bottom also rests 0.8 cm above the chassis bottom; limits shifted by the same amount so
+       the world-frame travel of the stack is unchanged -->
+  <xacro:property name="inner_mast_z" value="-0.0318"/>
+  <xacro:property name="inner_lower" value="-0.006"/>
+  <xacro:property name="inner_upper" value="0.2836"/>
+  <!-- forks (carriage). 0.0736 cancels the outer and inner mast drops so the forks keep their height at rest -->
+  <xacro:property name="forks_z" value="0.0736"/>
   <xacro:property name="forks_mass" value="0.15"/>
   <xacro:property name="forks_com" value="0.0178 0.0097 0.0196"/>
-  <xacro:property name="forks_lower" value="-0.01"/>
-  <xacro:property name="forks_upper" value="0.10"/>
+  <xacro:property name="forks_lower" value="-0.044"/>
+  <xacro:property name="forks_upper" value="0.0664"/>
   <xacro:property name="back_origin"  value="0.0056 0.01255 0.025"/>
   <xacro:property name="back_size"    value="0.0112 0.1087 0.0417"/>

File: src/puzzlebot_description/urdf/puzzlebot.urdf.xacro (robot description, xacro)
@@ -211,5 +211,5 @@
     <parent link="${prefix}outer_mast_link"/>
     <child  link="${prefix}inner_mast_link"/>
-    <origin xyz="0 0 0" rpy="0 0 0"/>
+    <origin xyz="0 0 ${inner_mast_z}" rpy="0 0 0"/>
     <axis xyz="0 0 1"/>
     <limit lower="${inner_lower}" upper="${inner_upper}" effort="10" velocity="0.05"/>
