Commit message: syntax fix to kalman node and xacro opti fm

File: src/puzzlebot_description/urdf/puzzlebot.urdf.xacro (robot description, xacro)
@@ -138,5 +138,5 @@
   </joint>
 <!-- camera -->
-  <link name="${prefix}camera">
+  <link name="${prefix}camera_link">
     <visual>
       <origin xyz="0 0 0" rpy="0 0 ${PI}"/>
@@ -155,7 +155,4 @@
       <origin xyz="0 0 0" rpy="0 0 0"/>
       <mass value="${camera_mass}"/>
-      <!--
-        Inercias calculadas con la geometría real de la caja.
-      -->
       <xacro:box_inertia
         m="${camera_mass}"
@@ -167,10 +164,18 @@
   <joint name="${prefix}chassis_to_camera" type="fixed">
     <parent link="${prefix}chassis"/>
-    <child  link="${prefix}camera"/>
+    <child  link="${prefix}camera_link"/>
     <origin xyz="${camera_x} ${camera_y} ${camera_z}"
-            rpy="${PI/2} ${PI} ${PI/2}"/>
+            rpy="0 0 0"/>
+  </joint>
+<!-- optical frame -->
+  <link name="${prefix}camera_color_optical_frame"/>
+  <joint name="${prefix}optical_frame" type="fixed">
+    <parent link="${prefix}camera_link"/>
+    <child  link="${prefix}camera_color_optical_frame"/>
+    <origin xyz="0.02 0 0"
+            rpy="-${PI/2} ${PI} -${PI/2}"/>
   </joint>
   <!-- lidar -->
-  <link name="${prefix}lidar">
+  <link name="${prefix}lidar_link">
     <visual>
       <origin xyz="0.07 -0.013 -0.04" rpy="${PI/2} 0 0"/>
@@ -197,5 +202,5 @@
   <joint name="${prefix}chassis_to_lidar" type="fixed">
     <parent link="${prefix}chassis"/>
-    <child  link="${prefix}lidar"/>
+    <child  link="${prefix}lidar_link"/>
     <origin xyz="${lidar_x} ${lidar_y} ${lidar_z}" rpy="0 0 ${PI}"/>
   </joint>

Commit message: forks joint added to robot state

File: src/puzzlebot_description/urdf/puzzlebot.urdf.xacro (robot description, xacro)
@@ -206,5 +206,5 @@
   </inertial>
 </link>
-<joint name="${prefix}inner_mast_joint" type="prismatic">
+<joint name="${prefix}inner_mast_joint" type="fixed">
   <parent link="${prefix}outer_mast_link"/>
   <child  link="${prefix}inner_mast_link"/>

Commit message: fixed GUI docker and rot lidar link

File: src/puzzlebot_description/urdf/puzzlebot.urdf.xacro (robot description, xacro)
@@ -156,5 +156,5 @@
     <parent link="${prefix}chassis_link"/>
     <child  link="${prefix}lidar_link"/>
-    <origin xyz="${lidar_x} ${lidar_y} ${lidar_z}" rpy="0 0 ${PI}"/>
+    <origin xyz="${lidar_x} ${lidar_y} ${lidar_z}" rpy="0 0 0"/>
   </joint>
     <!-- outer_mast  -->

Commit message: pkg refernce to meshes in xacro

File: src/puzzlebot_description/urdf/puzzlebot.urdf.xacro (robot description, xacro)
@@ -27,5 +27,6 @@
       <geometry>
    <!-- <mesh filename="../meshes3/puzzlebot_chassis_detailed.obj"/> -->
-        <mesh filename="file://${mesh_chassis}"/>
+        <!--<mesh filename="file://${mesh_chassis}"/> -->
+        <mesh filename="package://puzzlebot_description/meshes/puzzlebot_chassis_detailed.obj"/>
        <!-- <mesh filename="../meshes3/puzzlebot_chassis_detailed.obj"/> -->
       </geometry>
@@ -53,5 +54,7 @@
       <geometry>
    <!-- <mesh filename="../meshes3/puzzlebot_caster_wheel.obj"/> -->
-        <mesh filename="file://${caster_wheel}"/>
+        <!--<mesh filename="file://${caster_wheel}"/> -->
+        <!--<mesh filename="package://puzzlebot_description/meshes/puzzlebot_wheel.obj"/>-->
+        <mesh filename="package://puzzlebot_description/meshes/puzzlebot_caster_wheel.obj"/>
       </geometry>
       <material name="dark_grey"/>
@@ -80,5 +83,6 @@
       <geometry>
    <!-- <mesh filename="../meshes3/puzzlebot_wheel.obj"/> -->
-        <mesh filename="file://${mesh_wheel}"/>
+        <!--<mesh filename="file://${mesh_wheel}"/> -->
+        <mesh filename="package://puzzlebot_description/meshes/puzzlebot_wheel.obj"/>
       </geometry>
       <material name="orange"/>
@@ -111,5 +115,6 @@
       <geometry>
    <!-- <mesh filename="../meshes3/puzzlebot_wheel.obj"/> -->
-        <mesh filename="file://${mesh_wheel}"/>
+        <!--<mesh filename="file://${mesh_wheel}"/> -->
+        <mesh filename="package://puzzlebot_description/meshes/puzzlebot_wheel.obj"/>
       </geometry>
       <material name="orange"/>
@@ -164,5 +169,6 @@
     <geometry>
     <!-- <mesh filename="../meshes3/outer_mast.obj"/> -->
-      <mesh filename="file://${mesh_outer_mast}"/>
+      <!--<mesh filename="file://${mesh_outer_mast}"/> -->
+      <mesh filename="package://puzzlebot_description/meshes/outer_mast.obj"/>
     </geometry>
     <material name="black"/>
@@ -190,5 +196,6 @@
     <geometry>
  <!-- <mesh filename="../meshes3/inner_mast.obj"/> -->
-      <mesh filename="file://${mesh_inner_mast}"/>
+     <!-- <mesh filename="file://${mesh_inner_mast}"/>-->
+      <mesh filename="package://puzzlebot_description/meshes/inner_mast.obj"/>
     </geometry>
     <material name="black"/>
@@ -220,5 +227,6 @@
     <geometry>
   <!-- <mesh filename="../meshes3/forks.obj"/> -->
-      <mesh filename="file://${mesh_forks}"/>
+      <!--<mesh filename="file://${mesh_forks}"/>-->
+      <mesh filename="package://puzzlebot_description/meshes/forks.obj"/>
     </geometry>
     <material name="black"/>

Commit message: apriltag node py

File: src/puzzlebot_description/urdf/puzzlebot.urdf.xacro (robot description, xacro)
@@ -282,13 +282,12 @@
     <child  link="${prefix}camera_link"/>
     <origin xyz="${camera_x} ${camera_y} ${camera_z}"
-            rpy="0 0 0"/>
+            rpy="0 3.1416 3.1416"/>
   </joint>
 <!-- optical frame -->
   <link name="${prefix}camera_color_optical_frame"/>
-  <joint name="${prefix}optical_frame" type="fixed">
-    <parent link="${prefix}camera_link"/>
-    <child  link="${prefix}camera_color_optical_frame"/>
-    <origin xyz="0.0 0 0"
-            rpy="-${PI/2} -${PI/2} -${PI/2}"/>
-  </joint>
+<joint name="${prefix}optical_frame" type="fixed">
+  <parent link="${prefix}camera_link"/>
+  <child link="${prefix}camera_color_optical_frame"/>
+  <origin xyz="0.0 0 0" rpy="${-PI/2} 0 ${-PI/2}"/>
+</joint>
 </robot>

Commit message: lidar offset in yaw fixed

File: src/puzzlebot_description/urdf/puzzlebot.urdf.xacro (robot description, xacro)
@@ -142,5 +142,5 @@
   </joint>
   <!-- lidar -->
-  <link name="${prefix}lidar_link">
+  <link name="${prefix}laser">
     <collision>
       <origin xyz="0 0 0" rpy="0 0 0"/>
@@ -160,6 +160,6 @@
   <joint name="${prefix}chassis_to_lidar" type="fixed">
     <parent link="${prefix}chassis_link"/>
-    <child  link="${prefix}lidar_link"/>
-    <origin xyz="${lidar_x} ${lidar_y} ${lidar_z}" rpy="0 0 0"/>
+    <child  link="${prefix}laser"/>
+    <origin xyz="${lidar_x} ${lidar_y} ${lidar_z}" rpy="0 0 3.14"/>
   </joint>
     <!-- outer_mast  -->
