Commit message: fixed sim and odom bugs

File: src/puzzlebot_description/urdf/parameters.xacro (robot description, xacro)
@@ -24,7 +24,7 @@
   <xacro:property name="camera_height" value="0.06"/>
   <!-- camera position over the chassis-->
-  <xacro:property name="camera_x" value="0.09"/>
+  <xacro:property name="camera_x" value="0.08"/>
   <xacro:property name="camera_y" value="0.0"/>
-  <xacro:property name="camera_z" value="0.048"/>
+  <xacro:property name="camera_z" value="0.07"/>
   <xacro:property name="lidar_mass"   value="0.1"/>
   <xacro:property name="lidar_x"      value="0.05"/>

File: src/puzzlebot_description/urdf/puzzlebot.urdf.xacro (robot description, xacro)
@@ -173,5 +173,5 @@
     <parent link="${prefix}camera_link"/>
     <child  link="${prefix}camera_color_optical_frame"/>
-    <origin xyz="0.02 0 0"
+    <origin xyz="0.0 0 0"
             rpy="-${PI/2} 0 -${PI/2}"/>
   </joint>

Commit message: add real hw launch

File: src/puzzlebot_description/urdf/parameters.xacro (robot description, xacro)
@@ -6,5 +6,5 @@
   <xacro:property name="chassis_height" value="0.06"/>
   <xacro:property name="chassis_mass"   value="0.710"/>
-  <xacro:property name="wheel_radius"    value="0.05"/>
+  <xacro:property name="wheel_radius"    value="0.044"/>
   <xacro:property name="wheel_thickness" value="0.01"/>
   <xacro:property name="wheel_mass"      value="0.03"/>

Commit message: test for https

File: src/puzzlebot_description/urdf/parameters.xacro (robot description, xacro)
@@ -6,5 +6,5 @@
   <xacro:property name="chassis_height" value="0.06"/>
   <xacro:property name="chassis_mass"   value="0.710"/>
-  <xacro:property name="wheel_radius"    value="0.044"/>
+  <xacro:property name="wheel_radius"    value="0.051"/>
   <xacro:property name="wheel_thickness" value="0.01"/>
   <xacro:property name="wheel_mass"      value="0.03"/>

Commit message: optical frame fixed in xacro

File: src/puzzlebot_description/urdf/parameters.xacro (robot description, xacro)
@@ -27,5 +27,5 @@
   <xacro:property name="camera_height" value="0.06"/>
   <!-- camera position over the chassis /OVER THE FORKS-->
-  <xacro:property name="camera_x" value="0.0"/>
+  <xacro:property name="camera_x" value="0.02"/>
   <xacro:property name="camera_y" value="0.0"/>
   <xacro:property name="camera_z" value="0.10"/>

File: src/puzzlebot_description/urdf/puzzlebot.urdf.xacro (robot description, xacro)
@@ -289,5 +289,5 @@
   <parent link="${prefix}camera_link"/>
   <child link="${prefix}camera_color_optical_frame"/>
-  <origin xyz="0.0 0 0" rpy="${-PI/2} 0 ${-PI/2}"/>
+  <origin xyz="0.0 0 0" rpy="${PI/2} 0 ${PI/2}"/>
 </joint>
 </robot>

Commit message: extreinsec from fork to robot

File: src/puzzlebot_description/urdf/parameters.xacro (robot description, xacro)
@@ -15,5 +15,5 @@
 <!-- Distance from base link to the front edge of the chasis -->
   <xacro:property name="baselink_2_front"   value="0.09"/>
-  <xacro:property name="front_2_forklift"   value="0.03"/>
+  <xacro:property name="front_2_forklift"   value="0.05"/>
   <xacro:property name="caster_radius" value="0.0065"/>
   <xacro:property name="caster_mass"   value="0.012"/>
@@ -31,5 +31,5 @@
   <xacro:property name="camera_z" value="0.10"/>
   <xacro:property name="lidar_mass"   value="0.1"/>
-  <xacro:property name="lidar_x"      value="0.05"/>
+  <xacro:property name="lidar_x"      value="0.03"/>
   <xacro:property name="lidar_y"      value="0.0"/>
   <xacro:property name="lidar_z"      value="0.115"/>

Commit message: offset for camera

File: src/puzzlebot_description/urdf/parameters.xacro (robot description, xacro)
@@ -27,5 +27,5 @@
   <xacro:property name="camera_height" value="0.06"/>
   <!-- camera position over the chassis /OVER THE FORKS-->
-  <xacro:property name="camera_x" value="0.02"/>
+  <xacro:property name="camera_x" value="0.01"/>
   <xacro:property name="camera_y" value="0.0"/>
   <xacro:property name="camera_z" value="0.10"/>

File: src/puzzlebot_description/urdf/puzzlebot.urdf.xacro (robot description, xacro)
@@ -289,5 +289,5 @@
   <parent link="${prefix}camera_link"/>
   <child link="${prefix}camera_color_optical_frame"/>
-  <origin xyz="0.0 0 0" rpy="${PI/2} 0 ${PI/2}"/>
+  <origin xyz="0.05 0 0" rpy="${PI/2} 0 ${PI/2}"/>
 </joint>
 </robot>

Commit message: extrinssec of cam in new base

File: src/puzzlebot_description/urdf/parameters.xacro (robot description, xacro)
@@ -29,13 +29,14 @@
   <xacro:property name="camera_x" value="0.01"/>
   <xacro:property name="camera_y" value="0.0"/>
-  <xacro:property name="camera_z" value="0.10"/>
+  <xacro:property name="camera_z" value="0.15"/>
+  <!--<xacro:property name="forks_z" value="0.005"-->
   <xacro:property name="lidar_mass"   value="0.1"/>
   <xacro:property name="lidar_x"      value="0.03"/>
   <xacro:property name="lidar_y"      value="0.0"/>
   <xacro:property name="lidar_z"      value="0.115"/>
-  <!-- fork position over the chassis FRONT-->
+  <!-- fork position over the baseFRONT FRONT-->
   <xacro:property name="forks_x" value="${baselink_2_front + front_2_forklift}"/>
   <xacro:property name="forks_y" value="0.0"/>
-  <xacro:property name="forks_z" value="-0.04"/>
+  <xacro:property name="forks_z" value="0.005"/>
   <xacro:property name="forks_yaw" value= "0.0"/>
 <xacro:property name="mast_height"      value="0.169"/>

File: src/puzzlebot_description/urdf/puzzlebot.urdf.xacro (robot description, xacro)
@@ -187,5 +187,5 @@
 </link>
 <joint name="${prefix}outer_mast_joint" type="fixed">
-  <parent link="${prefix}chassis_link"/>
+  <parent link="${prefix}base_footprint"/>
   <child  link="${prefix}outer_mast_link"/>
   <origin xyz="${forks_x} ${forks_y} ${forks_z}" rpy="0 0 0"/>
@@ -257,5 +257,5 @@
   <origin xyz="0 0 0" rpy="0 0 0"/>
   <axis xyz="0 0 1"/>
-  <limit lower="0.0" upper="${fork_travel}" effort="50" velocity="0.1"/>
+  <limit lower="0.0" upper="${fork_travel}" effort="50" velocity="0.03"/>
   <dynamics damping="1.0" friction="0.5"/>
 </joint>
